Commit message: added tool joint axis

File: robot.URDF (robot description, URDF)
Before this commit: robot abb_irb120_3_58, 8 links, 7 joints
Joints:
- joint joint6-tool0: axis (none) -> 0 1 0

Commit message: ikpy bugs fixed

File: robot.URDF (robot description, URDF)
Before this commit: robot abb_irb120_3_58, 8 links, 7 joints
Links:
- removed link tool0
Joints:
- removed joint joint6-tool0
